Commit message: SLAM

File: pbl_launch/urdf/pbl.urdf.xacro (robot description, xacro)
@@ -3,10 +3,10 @@
   <xacro:property name="body_length" value="0.45"/>
   <xacro:property name="body_width" value="0.45"/>
-  <xacro:property name="body_height" value="0.08"/>
+  <xacro:property name="body_height" value="0.015"/>
   <xacro:property name="wheel_radius" value="0.05"/>
   <xacro:property name="wheel_width" value="0.01"/>
-  <xacro:property name="rear_wheel_from_rear_edge" value="0.085"/>
-  <xacro:property name="rear_wheel_x" value="${-body_length / 2.0 + rear_wheel_from_rear_edge}"/>
-  <xacro:property name="rear_wheel_y" value="${body_width / 2.0 + wheel_width / 2.0}"/>
+  <xacro:property name="wheel_separation" value="0.46"/>
+  <xacro:property name="base_center_offset" value="${body_length / 2.0 - 0.085}"/>
+  <xacro:property name="rear_wheel_y" value="${wheel_separation / 2.0}"/>
   <xacro:property name="rear_wheel_z" value="${wheel_radius}"/>
   <material name="body_gray">
@@ -23,5 +23,5 @@
     </inertial>
     <visual>
-      <origin xyz="0 0 ${wheel_radius + body_height / 2.0}" rpy="0 0 0"/>
+      <origin xyz="${base_center_offset} 0 ${wheel_radius + body_height / 2.0}" rpy="0 0 0"/>
       <geometry>
         <box size="${body_length} ${body_width} ${body_height}"/>
@@ -30,5 +30,5 @@
     </visual>
     <collision>
-      <origin xyz="0 0 ${wheel_radius + body_height / 2.0}" rpy="0 0 0"/>
+      <origin xyz="${base_center_offset} 0 ${wheel_radius + body_height / 2.0}" rpy="0 0 0"/>
       <geometry>
         <box size="${body_length} ${body_width} ${body_height}"/>
@@ -40,5 +40,5 @@
     <parent link="base_link"/>
     <child link="unilidar_lidar"/>
-    <origin xyz="${body_length / 2.0} 0 0" rpy="0 0 0"/>
+    <origin xyz="${body_length / 2.0 + base_center_offset} 0 ${wheel_radius + body_height / 2.0}" rpy="0 0 0"/>
   </joint>
   <link name="unilidar_imu"/>
@@ -76,5 +76,5 @@
     </joint>
   </xacro:macro>
-  <xacro:drive_wheel name="joint0" x="${rear_wheel_x}" y="${-rear_wheel_y}"/>
-  <xacro:drive_wheel name="joint1" x="${rear_wheel_x}" y="${+rear_wheel_y}"/>
+  <xacro:drive_wheel name="joint0" x="0.0" y="${-rear_wheel_y}"/>
+  <xacro:drive_wheel name="joint1" x="0.0" y="${rear_wheel_y}"/>
 </robot>

Commit message: fix some

File: pbl_launch/urdf/pbl.urdf.xacro (robot description, xacro)
@@ -4,4 +4,6 @@
   <xacro:property name="body_width" value="0.45"/>
   <xacro:property name="body_height" value="0.015"/>
+  <xacro:property name="pc_height" value="0.5"/>
+  <xacro:property name="pc_width" value="0.1"/>
   <xacro:property name="wheel_radius" value="0.05"/>
   <xacro:property name="wheel_width" value="0.01"/>
@@ -12,4 +14,7 @@
   <material name="body_gray">
     <color rgba="0.85 0.85 0.85 1.0"/>
+  </material>
+  <material name="pc_black">
+    <color rgba="0.08 0.08 0.08 1.0"/>
   </material>
   <material name="wheel_black">
@@ -36,4 +41,18 @@
     </collision>
   </link>
+  <link name="pc">
+    <visual>
+      <origin xyz="0 0 ${pc_height / 2.0}" rpy="0 0 0"/>
+      <geometry>
+        <box size="${pc_width} ${body_width} ${pc_height}"/>
+      </geometry>
+      <material name="pc_black"/>
+    </visual>
+  </link>
+  <joint name="base_link_to_pc" type="fixed">
+    <parent link="base_link"/>
+    <child link="pc"/>
+    <origin xyz="-0.04 0 ${wheel_radius + body_height}" rpy="0 0 0"/>
+  </joint>
   <link name="unilidar_lidar"/>
   <joint name="base_link_to_unilidar_lidar" type="fixed">

Commit message: add lidar filter

File: pbl_launch/urdf/pbl.urdf.xacro (robot description, xacro)
@@ -59,5 +59,5 @@
     <parent link="base_link"/>
     <child link="unilidar_lidar"/>
-    <origin xyz="${body_length / 2.0 + base_center_offset} 0 ${wheel_radius + body_height / 2.0}" rpy="0 0 0"/>
+    <origin xyz="${body_length / 2.0 + base_center_offset} 0 ${wheel_radius + body_height / 2.0}" rpy="0 0 0.3"/>
   </joint>
   <link name="unilidar_imu"/>

Commit message: 動く

File: pbl_launch/urdf/pbl.urdf.xacro (robot description, xacro)
@@ -59,5 +59,5 @@
     <parent link="base_link"/>
     <child link="unilidar_lidar"/>
-    <origin xyz="${body_length / 2.0 + base_center_offset} 0 ${wheel_radius + body_height / 2.0}" rpy="0 0 0.3"/>
+    <origin xyz="${body_length / 2.0 + base_center_offset} 0 ${wheel_radius + body_height / 2.0}" rpy="0 0 0.3926990816975"/>
   </joint>
   <link name="unilidar_imu"/>
